Commit message: update to Cartpole++ and SB domain extension

File: worlds/wsu/generator/models/ground_cart.urdf (robot description, URDF)
Before this commit: robot ground, 3 links, 2 joints
Links:
- link cart: mass 1 -> 1.0
- link pole: mass 1 -> 0.1
Joints:
- joint ground_to_cart: origin xyz=0.0 0.0 0.0 -> xyz=0.0 0.0 0.0 rpy=0.0 0.0 0.0

Commit message: working non-novel agent

File: worlds/wsu/generator/models/ground_cart.urdf (robot description, URDF)
Before this commit: robot ground, 3 links, 2 joints
Links:
- link ground: geometry collision box size=0.01 0.01 0.01; visual box size=0.1 0.1 0.3

Commit message: bringing it up to scratch

File: worlds/wsu/generator/models/ground_cart.urdf (robot description, URDF)
Before this commit: robot ground, 3 links, 2 joints
Links:
- link ground: geometry visual box size=0.1 0.1 0.3
- link pole: geometry collision cylinder length=1.0 radius=0.03; visual cylinder length=1.0 radius=0.03
Joints:
- joint pole_to_cart: origin xyz=0.0 0.0 0.2 -> xyz=0.0 0.0 0.2 rpy=0 0 0

File: worlds/wsu/generator/models/m4/block.urdf (robot description, URDF)
Before this commit: robot block, 1 links, 0 joints
Links:
- link block: geometry collision sphere radius=1.0; visual sphere radius=1.0

File: worlds/wsu/generator/models/walls.urdf (robot description, URDF)
Before this commit: robot wall, 6 links, 5 joints
Links:
- link wall5: geometry collision box size=10.1 10.1 0.1; visual box size=10.1 10.1 0.1
- link wall6: geometry collision box size=10.1 10.1 0.1; visual box size=10.1 10.1 0.1
